File: secondorderbasic/secondorderbasic-backups/secondorderbasic-2025-05-27_163612/_autosave-secondorderbasic.kicad_pcb (KiCad board)
At the start: 2 copper layers, 72 x 71 mm, 11 parts, among them U1 OP1177ARM

Commit message: testagain
Parts:
- removed R5: 0, Resistor_SMD:R_0603_1608Metric
- R3, R4: footprint Resistor_SMD:R_1020_2550Metric -> Resistor_SMD:R_0402_1005Metric
- moved R2 3.95 mm to (112.0, 106.0)
- moved R4 2.36 mm to (118.3, 109.8)
- moved R3 2.12 mm to (112.5, 103.0), turned to -90 degrees
Connections:
- C2 pad 1: /positivefeedback -> /negativefeedback
- C2 pad 2: /negativefeedback -> /positivefeedback
- R1 pad 1: /positivefeedback -> /negativefeedback
- R2 pad 2: /positivefeedback -> /negativefeedback
- R3 pad 2: /negativefeedback -> /positivefeedback
- U1 pad 6: /negativefeedback -> /positivefeedback
- U1 pad 7: Net-(U1-V+) -> Net-(BT1-+)
Routing:
- net Net-(BT3-+): track 44.9 -> 0.64 mm
- net Net-(BT1-+): track 45.1 -> 2.28 mm
- net Net-(U1-+): track 18.6 -> 1.39 mm
- net Net-(BT2-+): track 15.3 -> 0.04 mm
- net /negativefeedback: track 20.8 -> 6.06 mm
- net Net-(U1-V+): track 3.88 -> 0.00 mm
- net Net-(U1--): track 14.9 -> 14.0 mm
- net /positivefeedback: track 3.62 -> 2.87 mm
