File: secondorderbasic/secondorderbasic-backups/secondorderbasic-2025-05-27_163612/secondorderbasic.kicad_pcb (KiCad board)
At the start: 2 copper layers, 72 x 71 mm, 11 parts, among them U1 OP1177ARM

Commit message: testagain
Parts:
- removed R5: 0, Resistor_SMD:R_0603_1608Metric
- moved R3 2.69 mm to (108.5, 103.5), turned to -90 degrees
Connections:
- C2 pad 1: /positivefeedback -> /negativefeedback
- C2 pad 2: /negativefeedback -> /positivefeedback
- R1 pad 1: /positivefeedback -> /negativefeedback
- R2 pad 2: /positivefeedback -> /negativefeedback
- R3 pad 2: /negativefeedback -> /positivefeedback
- U1 pad 6: /negativefeedback -> /positivefeedback
- U1 pad 7: Net-(U1-V+) -> Net-(BT1-+)
Routing:
- net /negativefeedback: track 20.8 -> 1.69 mm
- net GND: track 43.6 -> 26.0 mm
- net Net-(U1-+): track 18.6 -> 1.39 mm
- net Net-(BT2-+): track 15.3 -> 30.0 mm
- net Net-(U1--): track 14.9 -> 23.6 mm
- net Net-(BT3-+): track 44.9 -> 36.3 mm
- net Net-(BT1-+): track 45.1 -> 49.9 mm
- net Net-(U1-V+): track 3.88 -> 0.00 mm
- net /positivefeedback: track 3.62 -> 0.00 mm
